Commit message: CLIK not finished

File: robots/models/GEN3-LITE.urdf (robot description, URDF)
Before this commit: robot KR7108-URDF, 8 links, 7 joints
Links:
- removed link DUMMY
- removed link END_EFFECTOR
- added link GRIPPER_FRAME, mass 0.1395; collision mesh filename=meshes/GRIPPER_FRAME.STL
- added link LEFT_FINGER_DIST, mass 0.010748; collision mesh filename=meshes/LEFT_FINGER_DIST.STL
- added link LEFT_FINGER_PROX, mass 0.018385; collision mesh filename=meshes/LEFT_FINGER_PROX.STL
- added link RIGHT_FINGER_DIST, mass 0.010748; collision mesh filename=meshes/RIGHT_FINGER_DIST.STL
- added link RIGHT_FINGER_PROX, mass 0.018385; collision mesh filename=meshes/RIGHT_FINGER_PROX.STL
- link ARM: geometry collision mesh filename=meshes/ARM.STL
- link BASE: geometry collision mesh filename=meshes/BASE.STL
- link FOREARM: geometry collision mesh filename=meshes/FOREARM.STL
- link LOWER_WRIST: geometry collision mesh filename=meshes/LOWER_WRIST.STL
- link SHOULDER: geometry collision mesh filename=meshes/SHOULDER.STL
- link UPPER_WRIST: geometry collision mesh filename=meshes/UPPER_WRIST.STL
Joints:
- removed joint END_EFFECTOR
- removed joint J0
- removed joint J1
- removed joint J2
- removed joint J3
- removed joint J4
- removed joint J5
- added joint 0: type revolute, parent BASE, child SHOULDER, origin xyz=0 0 0.12825 rpy=0 0 0, axis 0 0 1, limit lower=-2.76 upper=2.76 effort=10 velocity=0.35
- added joint 1: type revolute, parent SHOULDER, child ARM, origin xyz=0 -0.03 0.115 rpy=1.5708 0 0, axis 0 0 1, limit lower=-2.76 upper=2.76 effort=14 velocity=0.35
- added joint 2: type revolute, parent ARM, child FOREARM, origin xyz=0 0.28 0 rpy=-3.1416 0 0, axis 0 0 1, limit lower=-2.76 upper=2.76 effort=10 velocity=0.35
- added joint 3: type revolute, parent FOREARM, child LOWER_WRIST, origin xyz=0 -0.14 0.02 rpy=1.5708 0 0, axis 0 0 1, limit lower=-2.67 upper=2.67 effort=7 velocity=0.35
- added joint 4: type revolute, parent LOWER_WRIST, child UPPER_WRIST, origin xyz=0.0285 0 0.105 rpy=0 1.5708 0, axis 0 0 1, limit lower=-2.67 upper=2.67 effort=7 velocity=0.35
- added joint 5: type revolute, parent UPPER_WRIST, child GRIPPER_FRAME, origin xyz=-0.105 0 0.0285 rpy=0 -1.5708 0, axis 0 0 1, limit lower=-2.67 upper=2.67 effort=7 velocity=0.35
- added joint LEFT_BOTTOM: type fixed, parent GRIPPER_FRAME, child LEFT_FINGER_PROX, origin xyz=0 0.0305 0.070003 rpy=0 1.5708 0, axis 0 0 1, limit lower=-0.96 upper=0.09 effort=1000 velocity=1000
- added joint LEFT_TIP: type fixed, parent LEFT_FINGER_PROX, child LEFT_FINGER_DIST, origin xyz=-0.045636 -0.020423 6.9901E-05 rpy=0 0 0, axis 0 0 -1, limit lower=-0.21 upper=1.03 effort=1000 velocity=1000
- added joint RIGHT_BOTTOM: type fixed, parent GRIPPER_FRAME, child RIGHT_FINGER_PROX, origin xyz=0 -0.030501 0.070003 rpy=0 1.5708 0, axis 0 0 1, limit lower=-0.09 upper=0.96 effort=1000 velocity=1000
- added joint RIGHT_TIP: type fixed, parent RIGHT_FINGER_PROX, child RIGHT_FINGER_DIST, origin xyz=-0.045636 0.020423 0 rpy=0 0 0, axis 0 0 1, limit lower=-1.03 upper=0.21 effort=1000 velocity=1000
